File: PicoFlasherPlus.kicad_sch (KiCad schematic)
At the start: 4 parts, among them J1 1x7 Pin Header, SW1 SW_DIP_x01, U1 Pico, U2 TS3A27518EPW

Commit message: Update
Parts:
- added R1, R2: 10k, Resistor_SMD:R_0805_2012Metric_Pad1.20x1.40mm_HandSolder, symbol Device:R_US
- J1: footprint Connector_PinHeader_1.00mm:PinHeader_1x07_P1.00mm_Horizontal -> Connector_PinHeader_2.54mm:PinHeader_1x07_P2.54mm_Horizontal
Connections:
- net at SW1.2: now also U2.14 (IN2), U2.24 (IN1), R1.1; no longer U2.20 (~{EN})
- new net: R2.1, U2.20 (~{EN})
- new net GND: R1.2, R2.2
Changed lines of the file:
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@@
 (kicad_sch (version 20211123) (generator eeschema)
   (paper "A4")
+  (junction (at 80.01 121.92) (diameter 0) (color 0 0 0 0)
+  )
+  (junction (at 80.01 124.46) (diameter 0) (color 0 0 0 0)
+  )
   (junction (at 142.24 93.98) (diameter 0) (color 0 0 0 0)
   )
@@
     (stroke (width 0) (type default) (color 0 0 0 0))
   )
+  (wire (pts (xy 80.01 124.46) (xy 80.01 134.62))
+    (stroke (width 0) (type default) (color 0 0 0 0))
+  )
   (wire (pts (xy 165.1 101.6) (xy 160.02 101.6))
     (stroke (width 0) (type default) (color 0 0 0 0))
   )
+  (wire (pts (xy 90.17 142.24) (xy 90.17 151.13))
+    (stroke (width 0) (type default) (color 0 0 0 0))
+  )
   (wire (pts (xy 124.46 99.06) (xy 107.95 99.06))
     (stroke (width 0) (type default) (color 0 0 0 0))
@@
     (stroke (width 0) (type default) (color 0 0 0 0))
   )
-  (wire (pts (xy 80.01 113.03) (xy 80.01 116.84))
+  (wire (pts (xy 80.01 113.03) (xy 80.01 121.92))
+    (stroke (width 0) (type default) (color 0 0 0 0))
+  )
+  (wire (pts (xy 80.01 142.24) (xy 80.01 151.13))
     (stroke (width 0) (type default) (color 0 0 0 0))
   )
@@
     (stroke (width 0) (type default) (color 0 0 0 0))
   )
+  (wire (pts (xy 124.46 121.92) (xy 80.01 121.92))
+    (stroke (width 0) (type default) (color 0 0 0 0))
+  )
   (wire (pts (xy 120.65 158.75) (xy 138.43 158.75))
     (stroke (width 0) (type default) (color 0 0 0 0))
@@
     (stroke (width 0) (type default) (color 0 0 0 0))
   )
+  (wire (pts (xy 80.01 124.46) (xy 80.01 121.92))
+    (stroke (width 0) (type default) (color 0 0 0 0))
+  )
   (wire (pts (xy 113.03 166.37) (xy 138.43 166.37))
     (stroke (width 0) (type default) (color 0 0 0 0))
@@
     (stroke (width 0) (type default) (color 0 0 0 0))
   )
+  (wire (pts (xy 90.17 134.62) (xy 90.17 116.84))
+    (stroke (width 0) (type default) (color 0 0 0 0))
+  )
   (wire (pts (xy 124.46 54.61) (xy 107.95 54.61))
     (stroke (width 0) (type default) (color 0 0 0 0))
@@
     (stroke (width 0) (type default) (color 0 0 0 0))
   )
+  (wire (pts (xy 124.46 124.46) (xy 80.01 124.46))
+    (stroke (width 0) (type default) (color 0 0 0 0))
+  )
   (wire (pts (xy 123.19 156.21) (xy 138.43 156.21))
     (stroke (width 0) (type default) (color 0 0 0 0))
@@
     (stroke (width 0) (type default) (color 0 0 0 0))
   )
+  (wire (pts (xy 90.17 116.84) (xy 124.46 116.84))
+    (stroke (width 0) (type default) (color 0 0 0 0))
+  )
   (wire (pts (xy 194.31 127) (xy 194.31 85.09))
     (stroke (width 0) (type default) (color 0 0 0 0))
@@
   )
   (wire (pts (xy 107.95 99.06) (xy 107.95 171.45))
-    (stroke (width 0) (type default) (color 0 0 0 0))
-  )
-  (wire (pts (xy 80.01 116.84) (xy 124.46 116.84))
     (stroke (width 0) (type default) (color 0 0 0 0))
   )
@@
     (pin "9")
   )
+  (symbol (lib_id "power:GND") (at 80.01 151.13 0) (unit 1)
+    (in_bom yes) (on_board yes) (fields_autoplaced)
+    (property "Reference" "#PWR0101" (id 0) (at 80.01 157.48 0)
+      (effects (font (size 1.27 1.27)) hide)
+    )
+    (property "Value" "GND" (id 1) (at 80.01 156.21 0))
+    (property "Footprint" "" (id 2) (at 80.01 151.13 0)
+      (effects (font (size 1.27 1.27)) hide)
+    )
+    (property "Datasheet" "" (id 3) (at 80.01 151.13 0)
+      (effects (font (size 1.27 1.27)) hide)
+    )
+    (pin "1")
+  )
+  (symbol (lib_id "Device:R_US") (at 80.01 138.43 0) (unit 1)
+    (in_bom yes) (on_board yes) (fields_autoplaced)
+    (property "Reference" "R1" (id 0) (at 82.55 137.1599 0)
+      (effects (font (size 1.27 1.27)) (justify left))
+    )
+    (property "Value" "10k" (id 1) (at 82.55 139.6999 0)
+      (effects (font (size 1.27 1.27)) (justify left))
+    )
+    (property "Footprint" "Resistor_SMD:R_0805_2012Metric_Pad1.20x1.40mm_HandSolder" (id 2) (at 81.026 138.684 90)
+      (effects (font (size 1.27 1.27)) hide)
+    )
+    (property "Datasheet" "~" (id 3) (at 80.01 138.43 0)
+      (effects (font (size 1.27 1.27)) hide)
+    )
+    (pin "1")
+    (pin "2")
+  )
   (symbol (lib_id "Connector:Conn_01x07_Male") (at 143.51 163.83 180) (unit 1)
     (in_bom yes) (on_board yes)
@@
       (effects (font (size 1.27 1.27)) (justify right))
     )
-    (property "Footprint" "Connector_PinHeader_1.00mm:PinHeader_1x07_P1.00mm_Horizontal" (id 2) (at 143.51 163.83 0)
+    (property "Footprint" "Connector_PinHeader_2.54mm:PinHeader_1x07_P2.54mm_Horizontal" (id 2) (at 143.51 163.83 0)
       (effects (font (size 1.27 1.27)) hide)
     )
@@
     (pin "6")
     (pin "7")
+  )
+  (symbol (lib_id "power:GND") (at 90.17 151.13 0) (unit 1)
+    (in_bom yes) (on_board yes) (fields_autoplaced)
+    (property "Reference" "#PWR0102" (id 0) (at 90.17 157.48 0)
+      (effects (font (size 1.27 1.27)) hide)
+    )
+    (property "Value" "GND" (id 1) (at 90.17 156.21 0))
+    (property "Footprint" "" (id 2) (at 90.17 151.13 0)
+      (effects (font (size 1.27 1.27)) hide)
+    )
+    (property "Datasheet" "" (id 3) (at 90.17 151.13 0)
+      (effects (font (size 1.27 1.27)) hide)
+    )
+    (pin "1")
   )
   (symbol (lib_id "Analog_Switch:TS3A27518EPW") (at 142.24 114.3 0) (unit 1)
@@
     (pin "9")
   )
+  (symbol (lib_id "Device:R_US") (at 90.17 138.43 0) (unit 1)
+    (in_bom yes) (on_board yes) (fields_autoplaced)
+    (property "Reference" "R2" (id 0) (at 92.71 137.1599 0)
+      (effects (font (size 1.27 1.27)) (justify left))
+    )
+    (property "Value" "10k" (id 1) (at 92.71 139.6999 0)
+      (effects (font (size 1.27 1.27)) (justify left))
+    )
+    (property "Footprint" "Resistor_SMD:R_0805_2012Metric_Pad1.20x1.40mm_HandSolder" (id 2) (at 91.186 138.684 90)
+      (effects (font (size 1.27 1.27)) hide)
+    )
+    (property "Datasheet" "~" (id 3) (at 90.17 138.43 0)
+      (effects (font (size 1.27 1.27)) hide)
+    )
+    (pin "1")
+    (pin "2")
+  )
   (sheet_instances
     (path "/" (page "1"))
   )
   (symbol_instances
+    (path "/3732ff5b-0966-4276-a9a7-c8f0c859ad0f"
+      (reference "#PWR0101") (unit 1) (value "GND") (footprint "")
+    )
+    (path "/c22a4634-f003-49ab-a381-70d4add2c8e8"
+      (reference "#PWR0102") (unit 1) (value "GND") (footprint "")
+    )
     (path "/c0e4767f-7351-4a9d-9273-7f9d136c8459"
-      (reference "J1") (unit 1) (value "1x7 Pin Header") (footprint "Connector_PinHeader_1.00mm:PinHeader_1x07_P1.00mm_Horizontal")
+      (reference "J1") (unit 1) (value "1x7 Pin Header") (footprint "Connector_PinHeader_2.54mm:PinHeader_1x07_P2.54mm_Horizontal")
+    )
+    (path "/b94339ca-8934-45fe-9784-7ccc9b54e512"
+      (reference "R1") (unit 1) (value "10k") (footprint "Resistor_SMD:R_0805_2012Metric_Pad1.20x1.40mm_HandSolder")
+    )
+    (path "/f6e53718-3b81-4e4f-b54d-4514f5ff76e0"
+      (reference "R2") (unit 1) (value "10k") (footprint "Resistor_SMD:R_0805_2012Metric_Pad1.20x1.40mm_HandSolder")
     )
     (path "/065fee51-2c96-4a41-88bd-f88c07468bde"
